Commit message: On branch maps  Changes to be committed: 	modified:   launch/hmap.launch 	modified:   scripts/ackerman_6_wheels.py 	modified:   urdf/curiosity_mars_rover_properties.xacro

File: urdf/curiosity_mars_rover_properties.xacro (robot description, xacro)
@@ -41,5 +41,5 @@
 	<xacro:property name="suspension_steer_B_L_Y" value="0.21019"/>
 	<xacro:property name="suspension_steer_B_L_Z" value="0.450036"/>
-	<xacro:property name="suspension_steer_limit" value="0.6"/>
+	<xacro:property name="suspension_steer_limit" value="1.5708"/>
 	<xacro:property name="suspension_steer_effort" value="10000.0"/>
 	<xacro:property name="suspension_steer_velocity" value="10.0"/>
